Commit message: feat: 4 wheeled robot with skid steer drive

File: my_robot/urdf/my_robot.xacro (robot description, xacro)
@@ -2,4 +2,87 @@
 <robot xmlns:xacro="http://www.ros.org/wiki/xacro" name="my_robot">
   <xacro:include filename="$(find my_robot)/urdf/my_robot.gazebo" />
+  <!-- Scale the robot size to fit the environment -->
+  <xacro:property name="scale" value="1.0" />
+  <xacro:property name="chassis_width" value="${scale * 0.115}" />
+  <xacro:property name="chassis_length" value="${scale * 0.145}" />
+  <xacro:property name="chassis_height" value="${scale * 0.02}" />
+  <xacro:property name="chassis_mass" value="${scale * 0.1}" />
+  <xacro:property name="compute_width" value="${scale * 0.10}" />
+  <xacro:property name="compute_length" value="${scale * 0.12}" />
+  <xacro:property name="compute_height" value="${scale * 0.05}" />
+  <xacro:property name="compute_mass" value="${scale * 0.2}" />
+  <xacro:property name="camera_width" value="${scale * 0.02}" />
+  <xacro:property name="camera_length" value="${scale * 0.02}" />
+  <xacro:property name="camera_height" value="${scale * 0.02}" />
+  <xacro:property name="camera_mass" value="${scale * 0.02}" />
+  <xacro:property name="wheel_length" value="${scale * 0.03}" />
+  <xacro:property name="wheel_radius" value="${scale * 0.02}" />
+  <xacro:property name="wheel_mass" value="${scale * 1}" />
+  <xacro:property name="wheel_inertia" value="${scale * 1e-3}" />
+  <xacro:property name="wheel_separation" value="${scale * 0.12}" />
+  <xacro:property name="wheel_y_offset" value="${(chassis_width + wheel_length + 0.005)/2}" />
+  <xacro:property name="wheel_kp" value="1000000.0" />
+  <xacro:property name="wheel_kd" value="100.0" />
+  <xacro:property name="wheel_mu1" value="1" />
+  <xacro:property name="wheel_mu2" value="1" />
+  <xacro:property name="wheel_slip1" value="0.5" />
+  <xacro:property name="wheel_slip2" value="0" />
+ <!--All units in m-kg-s-radians unit system -->
+  <xacro:property name="M_PI" value="3.1415926535897931" />
+  <xacro:property name="M_PI_2" value="1.570796327" />
+  <xacro:property name="DEG_TO_RAD" value="0.017453293" />
+ <xacro:macro name="wheel" params="fb lr parent translateX translateY flipY"> <!--fb : front, back ; lr: left, right -->
+    <link name="${fb}_${lr}_wheel">
+      <visual>
+        <origin xyz="0 0 0" rpy="0 1.5707 1.5707" />
+        <geometry>
+          <cylinder length="${wheel_length}" radius="${wheel_radius}" />
+        </geometry>
+        <material name="DarkGray" />
+      </visual>
+      <collision>
+        <origin xyz="0 0 0" rpy="0 1.5707 1.5707" />
+        <geometry>
+          <cylinder length="${wheel_length}" radius="${wheel_radius}" />
+        </geometry>
+        <surface>
+          <friction>
+            <fdir1>1 0 0</fdir1>
+            <kp>${wheel_kp}</kp> <!-- kp and kd for rubber -->
+            <kd>${wheel_kd}</kd>
+            <mu>${wheel_mu1}</mu>
+            <mu2>${wheel_mu2}</mu2>
+            <slip1>${wheel_slip1}</slip1>
+            <slip2>${wheel_slip2}</slip2>
+          </friction>
+        </surface>
+      </collision>
+      <inertial>
+        <mass value="${wheel_mass}"/>
+        <origin xyz="0.0 0 0" rpy="0 1.5707 1.5707"/>
+        <inertia
+          ixx="${wheel_inertia}" ixy="0" ixz="0"
+          iyy="${wheel_inertia}" iyz="0"
+          izz="${wheel_inertia}" />
+      </inertial>
+    </link>
+    <joint name="${fb}_${lr}_wheel_joint" type="continuous">
+      <parent link="${parent}"/>
+      <child link="${fb}_${lr}_wheel"/>
+      <origin xyz="${translateX} ${translateY} 0" rpy="0 0 0" />
+      <axis xyz="0 1 0" rpy="0 0 0" />
+      <limit effort="100" velocity="100"/>
+      <joint_properties damping="0.0" friction="0.0"/>
+    </joint>
+  </xacro:macro>
+  <gazebo reference="camera">
+    <material>Gazebo/Black</material>
+  </gazebo>
+  <gazebo reference="compute">
+    <material>Gazebo/Green</material>
+  </gazebo>
+  <gazebo reference="chassis">
+    <material>Gazebo/Blue</material>
+  </gazebo>
   <link name="robot_footprint"/>
   <joint name="robot_footprint_joint" type="fixed">
@@ -11,5 +94,5 @@
   <link name="camera">
     <inertial>
-      <mass value=".1"/>
+      <mass value="${camera_mass}"/>
       <origin xyz="0 0 0" rpy="0 0 0"/>
       <inertia ixx="1e-6" ixy="0" ixz="0" iyy="1e-6" iyz="0" izz="1e-6"/>
@@ -18,5 +101,5 @@
       <origin xyz="0 0 0" rpy="0 0 0"/>
       <geometry>
-        <box size=".05 .05 .05"/>
+        <box size="${camera_length} ${camera_width} ${camera_height}"/>
       </geometry>
     </collision>
@@ -24,11 +107,8 @@
       <origin xyz="0 0 0" rpy="0 0 0"/>
       <geometry>
-        <box size=".05 .05 .05"/>
+        <box size="${camera_length} ${camera_width} ${camera_height}"/>
       </geometry>
     </visual>
   </link>
-  <gazebo reference="camera">
-    <material>Gazebo/Black</material>
-  </gazebo>
   <!-- lidar -->
   <link name="hokuyo">
@@ -51,55 +131,9 @@
     </visual>
   </link>
-  <!-- left wheel -->
-  <link name="left_wheel">
-    <inertial>
-      <mass value="5"/>
-      <origin xyz="0 0 0" rpy="0 1.5707 1.5707"/>
-      <inertia ixx="0.1" ixy="0" ixz="0" iyy="0.1" iyz="0" izz="0.1"/>
-    </inertial>
-    <collision>
-      <origin xyz="0 0 0" rpy="0 1.5707 1.5707"/>
-      <geometry>
-        <cylinder length="0.05" radius="0.1"/>
-      </geometry>
-    </collision>
-    <visual>
-      <origin xyz="0 0 0" rpy=" 0 1.5707 1.5707"/>
-      <geometry>
-        <cylinder length="0.05" radius="0.1"/>
-      </geometry>
-    </visual>
-  </link>
-  <gazebo reference="left_wheel">
-    <material>Gazebo/White</material>
-  </gazebo>
-  <!-- right wheel -->
-  <link name="right_wheel">
-    <inertial>
-      <mass value="5"/>
-      <origin xyz="0 0 0" rpy="0 1.5707 1.5707"/>
-      <inertia ixx="0.1" ixy="0" ixz="0" iyy="0.1" iyz="0" izz="0.1"/>
-    </inertial>
-    <collision>
-      <origin xyz="0 0 0" rpy="0 1.5707 1.5707"/>
-      <geometry>
-        <cylinder length="0.05" radius="0.1"/>
-      </geometry>
-    </collision>
-    <visual>
-      <origin xyz="0 0 0" rpy=" 0 1.5707 1.5707"/>
-      <geometry>
-        <cylinder length="0.05" radius="0.1"/>
-      </geometry>
-    </visual>
-  </link>
-  <gazebo reference="right_wheel">
-    <material>Gazebo/White</material>
-  </gazebo>
   <!--- chassis -->
   <link name="chassis">
     <pose>0 0 0.1 0 0 0</pose>
     <inertial>
-      <mass value="15.0"/>
+      <mass value="${chassis_mass}"/>
       <origin xyz="0.0 0 0" rpy=" 0 0 0"/>
       <inertia ixx="0.1" ixy="0" ixz="0" iyy="0.1" iyz="0" izz="0.1"/>
@@ -108,5 +142,5 @@
       <origin xyz="0 0 0" rpy=" 0 0 0"/>
       <geometry>
-        <box size=".4 .2 .1"/>
+        <box size="${chassis_length} ${chassis_width} ${chassis_height}"/>
       </geometry>
     </collision>
@@ -114,62 +148,50 @@
       <origin xyz="0 0 0" rpy=" 0 0 0"/>
       <geometry>
-        <box size=".4 .2 .1"/>
-      </geometry>
-    </visual>
-    <collision name="back_caster_collision">
-      <origin xyz="-0.15 0 -0.05" rpy=" 0 0 0"/>
-      <geometry>
-        <sphere radius="0.0499"/>
-      </geometry>
-    </collision>
-    <visual name="back_caster_visual">
-      <origin xyz="-0.15 0 -0.05" rpy=" 0 0 0"/>
-      <geometry>
-        <sphere radius="0.05"/>
-      </geometry>
-    </visual>
-    <collision name="front_caster_collision">
-      <origin xyz="0.15 0 -0.05" rpy=" 0 0 0"/>
-      <geometry>
-        <sphere radius="0.0499"/>
-      </geometry>
-    </collision>
-    <visual name="front_caster_visual">
-      <origin xyz="0.15 0 -0.05" rpy=" 0 0 0"/>
-      <geometry>
-        <sphere radius="0.05"/>
+        <box size="${chassis_length} ${chassis_width} ${chassis_height}"/>
       </geometry>
     </visual>
   </link>
-  <gazebo reference="chassis">
-    <material>Gazebo/Blue</material>
-  </gazebo>
-  <joint type="continuous" name="left_wheel_hinge">
-    <origin xyz="0 0.15 0" rpy="0 0 0"/>
-    <child link="left_wheel"/>
-    <parent link="chassis"/>
+  <!--- compute -->
+  <link name="compute">
+    <pose>0.01 0 0.03 0 0 0</pose>
+    <inertial>
+      <mass value="${compute_mass}"/>
+      <origin xyz="0.0 0 0" rpy=" 0 0 0"/>
+      <inertia ixx="0.1" ixy="0" ixz="0" iyy="0.1" iyz="0" izz="0.1"/>
+    </inertial>
+    <collision name="compute_collision">
+      <origin xyz="0 0 0" rpy=" 0 0 0"/>
+      <geometry>
+        <box size="${compute_length} ${compute_width} ${compute_height}"/>
+      </geometry>
+    </collision>
+    <visual name="chassis_visual">
+      <origin xyz="0 0 0" rpy=" 0 0 0"/>
+      <geometry>
+        <box size="${compute_length} ${compute_width} ${compute_height}"/>
+      </geometry>
+    </visual>
+  </link>
+  <joint type="fixed" name="camera_joint">
+    <origin xyz="${camera_length/2 + compute_length/2} 0 0" rpy="0 0 0"/>
+    <child link="camera"/>
+    <parent link="compute"/>
     <axis xyz="0 1 0" rpy="0 0 0"/>
-    <limit effort="10000" velocity="1000"/>
-    <dynamics damping="1.0" friction="1.0"/>
   </joint>
-  <joint type="continuous" name="right_wheel_hinge">
-    <origin xyz="0 -0.15 0" rpy="0 0 0"/>
-    <child link="right_wheel"/>
-    <parent link="chassis"/>
+  <joint type="fixed" name="hokuyo_joint">
+    <origin xyz="0 0 .07" rpy="0 0 0"/>
+    <child link="hokuyo"/>
+    <parent link="compute"/>
     <axis xyz="0 1 0" rpy="0 0 0"/>
-    <limit effort="10000" velocity="1000"/>
-    <dynamics damping="1.0" friction="1.0"/>
   </joint>
-  <joint type="fixed" name="camera_joint">
-    <origin xyz=".2 0 0" rpy="0 0 0"/>
-    <child link="camera"/>
+  <joint type="fixed" name="compute_joint">
+    <origin xyz="0 0 ${chassis_height/2 + compute_height/2}" rpy="0 0 0"/>
+    <child link="compute"/>
     <parent link="chassis"/>
     <axis xyz="0 1 0" rpy="0 0 0"/>
   </joint>
-  <joint type="fixed" name="hokuyo_joint">
-    <origin xyz=".15 0 .1" rpy="0 0 0"/>
-    <child link="hokuyo"/>
-    <parent link="chassis"/>
-    <axis xyz="0 1 0" rpy="0 0 0"/>
-  </joint>
+  <xacro:wheel fb="front" lr="right" parent="chassis" translateX="${wheel_separation/2}" translateY="-${wheel_y_offset}" flipY="1"/>
+  <xacro:wheel fb="front" lr="left" parent="chassis" translateX="${wheel_separation/2}" translateY="${wheel_y_offset}" flipY="1"/>
+  <xacro:wheel fb="back" lr="right" parent="chassis" translateX="-${wheel_separation/2}" translateY="-${wheel_y_offset}" flipY="1"/>
+  <xacro:wheel fb="back" lr="left" parent="chassis" translateX="-${wheel_separation/2}" translateY="${wheel_y_offset}" flipY="1"/>
 </robot>

Commit message: fix: linked lidar that was flying over the robot

File: my_robot/urdf/my_robot.xacro (robot description, xacro)
@@ -32,5 +32,5 @@
   <xacro:property name="M_PI_2" value="1.570796327" />
   <xacro:property name="DEG_TO_RAD" value="0.017453293" />
- <xacro:macro name="wheel" params="fb lr parent translateX translateY flipY"> <!--fb : front, back ; lr: left, right -->
+ <xacro:macro name="wheel" params="fb lr parent translateX translateY"> <!--fb : front, back ; lr: left, right -->
     <link name="${fb}_${lr}_wheel">
       <visual>
@@ -180,5 +180,5 @@
   </joint>
   <joint type="fixed" name="hokuyo_joint">
-    <origin xyz="0 0 .07" rpy="0 0 0"/>
+    <origin xyz="0 0 .02" rpy="0 0 0"/>
     <child link="hokuyo"/>
     <parent link="compute"/>
@@ -191,7 +191,7 @@
     <axis xyz="0 1 0" rpy="0 0 0"/>
   </joint>
-  <xacro:wheel fb="front" lr="right" parent="chassis" translateX="${wheel_separation/2}" translateY="-${wheel_y_offset}" flipY="1"/>
-  <xacro:wheel fb="front" lr="left" parent="chassis" translateX="${wheel_separation/2}" translateY="${wheel_y_offset}" flipY="1"/>
-  <xacro:wheel fb="back" lr="right" parent="chassis" translateX="-${wheel_separation/2}" translateY="-${wheel_y_offset}" flipY="1"/>
-  <xacro:wheel fb="back" lr="left" parent="chassis" translateX="-${wheel_separation/2}" translateY="${wheel_y_offset}" flipY="1"/>
+  <xacro:wheel fb="front" lr="right" parent="chassis" translateX="${wheel_separation/2}" translateY="-${wheel_y_offset}"/>
+  <xacro:wheel fb="front" lr="left" parent="chassis" translateX="${wheel_separation/2}" translateY="${wheel_y_offset}"/>
+  <xacro:wheel fb="back" lr="right" parent="chassis" translateX="-${wheel_separation/2}" translateY="-${wheel_y_offset}"/>
+  <xacro:wheel fb="back" lr="left" parent="chassis" translateX="-${wheel_separation/2}" translateY="${wheel_y_offset}"/>
 </robot>

Commit message: feat: robustness, stops in front of ball

File: my_robot/urdf/my_robot.xacro (robot description, xacro)
@@ -4,21 +4,21 @@
   <!-- Scale the robot size to fit the environment -->
   <xacro:property name="scale" value="1.0" />
-  <xacro:property name="chassis_width" value="${scale * 0.115}" />
-  <xacro:property name="chassis_length" value="${scale * 0.145}" />
+  <xacro:property name="chassis_width" value="${scale * 0.2}" />
+  <xacro:property name="chassis_length" value="${scale * 0.45}" />
   <xacro:property name="chassis_height" value="${scale * 0.02}" />
-  <xacro:property name="chassis_mass" value="${scale * 0.1}" />
+  <xacro:property name="chassis_mass" value="${scale * 0.2}" />
   <xacro:property name="compute_width" value="${scale * 0.10}" />
   <xacro:property name="compute_length" value="${scale * 0.12}" />
   <xacro:property name="compute_height" value="${scale * 0.05}" />
-  <xacro:property name="compute_mass" value="${scale * 0.2}" />
+  <xacro:property name="compute_mass" value="${scale * 0.1}" />
   <xacro:property name="camera_width" value="${scale * 0.02}" />
   <xacro:property name="camera_length" value="${scale * 0.02}" />
   <xacro:property name="camera_height" value="${scale * 0.02}" />
   <xacro:property name="camera_mass" value="${scale * 0.02}" />
-  <xacro:property name="wheel_length" value="${scale * 0.03}" />
-  <xacro:property name="wheel_radius" value="${scale * 0.02}" />
-  <xacro:property name="wheel_mass" value="${scale * 1}" />
+  <xacro:property name="wheel_length" value="${scale * 0.045}" />
+  <xacro:property name="wheel_radius" value="${scale * 0.05}" />
+  <xacro:property name="wheel_mass" value="${scale * .01}" />
   <xacro:property name="wheel_inertia" value="${scale * 1e-3}" />
-  <xacro:property name="wheel_separation" value="${scale * 0.12}" />
+  <xacro:property name="wheel_separation" value="${scale * 0.32}" />
   <xacro:property name="wheel_y_offset" value="${(chassis_width + wheel_length + 0.005)/2}" />
   <xacro:property name="wheel_kp" value="1000000.0" />
@@ -174,7 +174,7 @@
   </link>
   <joint type="fixed" name="camera_joint">
-    <origin xyz="${camera_length/2 + compute_length/2} 0 0" rpy="0 0 0"/>
+    <origin xyz="${chassis_length/2 - camera_length} 0 ${chassis_height/2 + camera_height/2}" rpy="0 0 0"/>
     <child link="camera"/>
-    <parent link="compute"/>
+    <parent link="chassis"/>
     <axis xyz="0 1 0" rpy="0 0 0"/>
   </joint>

Commit message: feat: improved stability

File: my_robot/urdf/my_robot.xacro (robot description, xacro)
@@ -7,5 +7,5 @@
   <xacro:property name="chassis_length" value="${scale * 0.45}" />
   <xacro:property name="chassis_height" value="${scale * 0.02}" />
-  <xacro:property name="chassis_mass" value="${scale * 0.2}" />
+  <xacro:property name="chassis_mass" value="${scale * 0.5}" />
   <xacro:property name="compute_width" value="${scale * 0.10}" />
   <xacro:property name="compute_length" value="${scale * 0.12}" />
@@ -18,5 +18,5 @@
   <xacro:property name="wheel_length" value="${scale * 0.045}" />
   <xacro:property name="wheel_radius" value="${scale * 0.05}" />
-  <xacro:property name="wheel_mass" value="${scale * .01}" />
+  <xacro:property name="wheel_mass" value="${scale * .05}" />
   <xacro:property name="wheel_inertia" value="${scale * 1e-3}" />
   <xacro:property name="wheel_separation" value="${scale * 0.32}" />

Commit message: feat: improved stability of steering

File: my_robot/urdf/my_robot.xacro (robot description, xacro)
@@ -7,5 +7,5 @@
   <xacro:property name="chassis_length" value="${scale * 0.45}" />
   <xacro:property name="chassis_height" value="${scale * 0.02}" />
-  <xacro:property name="chassis_mass" value="${scale * 0.5}" />
+  <xacro:property name="chassis_mass" value="${scale * 0.1}" />
   <xacro:property name="compute_width" value="${scale * 0.10}" />
   <xacro:property name="compute_length" value="${scale * 0.12}" />
@@ -23,5 +23,5 @@
   <xacro:property name="wheel_y_offset" value="${(chassis_width + wheel_length + 0.005)/2}" />
   <xacro:property name="wheel_kp" value="1000000.0" />
-  <xacro:property name="wheel_kd" value="100.0" />
+  <xacro:property name="wheel_kd" value="10.0" />
   <xacro:property name="wheel_mu1" value="1" />
   <xacro:property name="wheel_mu2" value="1" />
@@ -55,4 +55,6 @@
             <slip1>${wheel_slip1}</slip1>
             <slip2>${wheel_slip2}</slip2>
+            <maxVel>0.001</maxVel>
+            <minDepth>0</minDepth>
           </friction>
         </surface>

Commit message: feat: improved stability
* optimizations inspired by Drive Train Basics by Chris Hibner
  https://www.chiefdelphi.com/t/white-paper-discuss-drive-train-basics/46562

File: my_robot/urdf/my_robot.xacro (robot description, xacro)
@@ -4,5 +4,5 @@
   <!-- Scale the robot size to fit the environment -->
   <xacro:property name="scale" value="1.0" />
-  <xacro:property name="chassis_width" value="${scale * 0.2}" />
+  <xacro:property name="chassis_width" value="${scale * 0.45}" />
   <xacro:property name="chassis_length" value="${scale * 0.45}" />
   <xacro:property name="chassis_height" value="${scale * 0.02}" />
@@ -16,5 +16,5 @@
   <xacro:property name="camera_height" value="${scale * 0.02}" />
   <xacro:property name="camera_mass" value="${scale * 0.02}" />
-  <xacro:property name="wheel_length" value="${scale * 0.045}" />
+  <xacro:property name="wheel_length" value="${scale * 0.02}" />
   <xacro:property name="wheel_radius" value="${scale * 0.05}" />
   <xacro:property name="wheel_mass" value="${scale * .05}" />
@@ -188,5 +188,5 @@
   </joint>
   <joint type="fixed" name="compute_joint">
-    <origin xyz="0 0 ${chassis_height/2 + compute_height/2}" rpy="0 0 0"/>
+    <origin xyz="-${compute_height/2} 0 ${chassis_height/2 + compute_height/2}" rpy="0 0 0"/>
     <child link="compute"/>
     <parent link="chassis"/>

Commit message: feat: set initial position, reduced num particles

File: my_robot/urdf/my_robot.xacro (robot description, xacro)
@@ -20,12 +20,16 @@
   <xacro:property name="wheel_mass" value="${scale * .05}" />
   <xacro:property name="wheel_inertia" value="${scale * 1e-3}" />
-  <xacro:property name="wheel_separation" value="${scale * 0.32}" />
-  <xacro:property name="wheel_y_offset" value="${(chassis_width + wheel_length + 0.005)/2}" />
+  <xacro:property name="wheel_separation" value="${chassis_width + wheel_length + 2*0.005*scale}" />
+  <xacro:property name="wheel_base" value="${scale * 0.32}" />
+  <xacro:property name="wheel_y_offset" value="${wheel_separation/2}" />
   <xacro:property name="wheel_kp" value="1000000.0" />
   <xacro:property name="wheel_kd" value="10.0" />
+  <xacro:property name="wheel_fdir1" value="1 0 0" />
   <xacro:property name="wheel_mu1" value="1" />
   <xacro:property name="wheel_mu2" value="1" />
   <xacro:property name="wheel_slip1" value="0.5" />
   <xacro:property name="wheel_slip2" value="0" />
+  <xacro:property name="wheel_maxVel" value="0" />
+  <xacro:property name="wheel_minDepth" value="0.001" />
  <!--All units in m-kg-s-radians unit system -->
   <xacro:property name="M_PI" value="3.1415926535897931" />
@@ -48,5 +52,5 @@
         <surface>
           <friction>
-            <fdir1>1 0 0</fdir1>
+            <fdir1>${wheel_fdir1}</fdir1>
             <kp>${wheel_kp}</kp> <!-- kp and kd for rubber -->
             <kd>${wheel_kd}</kd>
@@ -55,6 +59,6 @@
             <slip1>${wheel_slip1}</slip1>
             <slip2>${wheel_slip2}</slip2>
-            <maxVel>0.001</maxVel>
-            <minDepth>0</minDepth>
+            <!--<maxVel>${wheel_maxVel}</maxVel>
+            <minDepth>${wheel_minDepth}</minDepth>-->
           </friction>
         </surface>
@@ -193,7 +197,7 @@
     <axis xyz="0 1 0" rpy="0 0 0"/>
   </joint>
-  <xacro:wheel fb="front" lr="right" parent="chassis" translateX="${wheel_separation/2}" translateY="-${wheel_y_offset}"/>
-  <xacro:wheel fb="front" lr="left" parent="chassis" translateX="${wheel_separation/2}" translateY="${wheel_y_offset}"/>
-  <xacro:wheel fb="back" lr="right" parent="chassis" translateX="-${wheel_separation/2}" translateY="-${wheel_y_offset}"/>
-  <xacro:wheel fb="back" lr="left" parent="chassis" translateX="-${wheel_separation/2}" translateY="${wheel_y_offset}"/>
+  <xacro:wheel fb="front" lr="right" parent="chassis" translateX="${wheel_base/2}" translateY="-${wheel_y_offset}"/>
+  <xacro:wheel fb="front" lr="left" parent="chassis" translateX="${wheel_base/2}" translateY="${wheel_y_offset}"/>
+  <xacro:wheel fb="back" lr="right" parent="chassis" translateX="-${wheel_base/2}" translateY="-${wheel_y_offset}"/>
+  <xacro:wheel fb="back" lr="left" parent="chassis" translateX="-${wheel_base/2}" translateY="${wheel_y_offset}"/>
 </robot>
