Commit message: fix: replaced robot with skid-steer-drive by  robot with simple differential drive in order to improvecontrol accuracy

File: my_robot/urdf/my_robot.xacro (robot description, xacro)
@@ -4,12 +4,8 @@
   <!-- Scale the robot size to fit the environment -->
   <xacro:property name="scale" value="1.0" />
-  <xacro:property name="chassis_width" value="${scale * 0.45}" />
-  <xacro:property name="chassis_length" value="${scale * 0.45}" />
-  <xacro:property name="chassis_height" value="${scale * 0.02}" />
+  <xacro:property name="chassis_width" value="${scale * 0.20}" />
+  <xacro:property name="chassis_length" value="${scale * 0.20}" />
+  <xacro:property name="chassis_height" value="${scale * 0.05}" />
   <xacro:property name="chassis_mass" value="${scale * 0.1}" />
-  <xacro:property name="compute_width" value="${scale * 0.10}" />
-  <xacro:property name="compute_length" value="${scale * 0.12}" />
-  <xacro:property name="compute_height" value="${scale * 0.05}" />
-  <xacro:property name="compute_mass" value="${scale * 0.1}" />
   <xacro:property name="camera_width" value="${scale * 0.02}" />
   <xacro:property name="camera_length" value="${scale * 0.02}" />
@@ -23,19 +19,24 @@
   <xacro:property name="wheel_base" value="${scale * 0.32}" />
   <xacro:property name="wheel_y_offset" value="${wheel_separation/2}" />
-  <xacro:property name="wheel_kp" value="1000000.0" />
-  <xacro:property name="wheel_kd" value="10.0" />
-  <xacro:property name="wheel_fdir1" value="1 0 0" />
-  <xacro:property name="wheel_mu1" value="1" />
-  <xacro:property name="wheel_mu2" value="1" />
-  <xacro:property name="wheel_slip1" value="0.5" />
-  <xacro:property name="wheel_slip2" value="0" />
-  <xacro:property name="wheel_maxVel" value="0" />
-  <xacro:property name="wheel_minDepth" value="0.001" />
+  <xacro:property name="caster_wheel_radius" value="${(wheel_radius - chassis_height/2)/2}"/>
+  <xacro:property name="caster_wheel_joint_offset" value="-${chassis_length/2-caster_wheel_radius}"/>
  <!--All units in m-kg-s-radians unit system -->
   <xacro:property name="M_PI" value="3.1415926535897931" />
   <xacro:property name="M_PI_2" value="1.570796327" />
   <xacro:property name="DEG_TO_RAD" value="0.017453293" />
- <xacro:macro name="wheel" params="fb lr parent translateX translateY"> <!--fb : front, back ; lr: left, right -->
-    <link name="${fb}_${lr}_wheel">
+  <xacro:macro name="sphere_inertia" params="m r">
+    <inertial>
+      <mass value="${m}"/>
+      <inertia ixx="${2.0*m*(r*r)/5.0}" ixy="0.0" ixz="0.0" iyy="${2.0*m*(r*r)/5.0}" iyz="0.0" izz="${2.0*m*(r*r)/5.0}"/>
+    </inertial>
+  </xacro:macro>
+<xacro:macro name="cylinder_inertia" params="m r h">
+    <inertial>
+      <mass value="${m}"/>
+      <inertia ixx="${m*(3*r*r+h*h)/12}" ixy = "0" ixz = "0" iyy="${m*(3*r*r+h*h)/12}" iyz = "0" izz="${m*r*r/2}"/>
+    </inertial>
+  </xacro:macro>
+ <xacro:macro name="wheel" params="lr parent translateX translateY"> <!--lr: left, right -->
+    <link name="${lr}_wheel">
       <visual>
         <origin xyz="0 0 0" rpy="0 1.5707 1.5707" />
@@ -50,30 +51,10 @@
           <cylinder length="${wheel_length}" radius="${wheel_radius}" />
         </geometry>
-        <surface>
-          <friction>
-            <fdir1>${wheel_fdir1}</fdir1>
-            <kp>${wheel_kp}</kp> <!-- kp and kd for rubber -->
-            <kd>${wheel_kd}</kd>
-            <mu>${wheel_mu1}</mu>
-            <mu2>${wheel_mu2}</mu2>
-            <slip1>${wheel_slip1}</slip1>
-            <slip2>${wheel_slip2}</slip2>
-            <!--<maxVel>${wheel_maxVel}</maxVel>
-            <minDepth>${wheel_minDepth}</minDepth>-->
-          </friction>
-        </surface>
       </collision>
-      <inertial>
-        <mass value="${wheel_mass}"/>
-        <origin xyz="0.0 0 0" rpy="0 1.5707 1.5707"/>
-        <inertia
-          ixx="${wheel_inertia}" ixy="0" ixz="0"
-          iyy="${wheel_inertia}" iyz="0"
-          izz="${wheel_inertia}" />
-      </inertial>
+      <xacro:cylinder_inertia m="10" r="${wheel_radius}" h="${wheel_length}"/>
     </link>
-    <joint name="${fb}_${lr}_wheel_joint" type="continuous">
+    <joint name="${lr}_wheel_joint" type="continuous">
       <parent link="${parent}"/>
-      <child link="${fb}_${lr}_wheel"/>
+      <child link="${lr}_wheel"/>
       <origin xyz="${translateX} ${translateY} 0" rpy="0 0 0" />
       <axis xyz="0 1 0" rpy="0 0 0" />
@@ -84,7 +65,4 @@
   <gazebo reference="camera">
     <material>Gazebo/Black</material>
-  </gazebo>
-  <gazebo reference="compute">
-    <material>Gazebo/Green</material>
   </gazebo>
   <gazebo reference="chassis">
@@ -158,25 +136,35 @@
     </visual>
   </link>
-  <!--- compute -->
-  <link name="compute">
-    <pose>0.01 0 0.03 0 0 0</pose>
-    <inertial>
-      <mass value="${compute_mass}"/>
-      <origin xyz="0.0 0 0" rpy=" 0 0 0"/>
-      <inertia ixx="0.1" ixy="0" ixz="0" iyy="0.1" iyz="0" izz="0.1"/>
-    </inertial>
-    <collision name="compute_collision">
-      <origin xyz="0 0 0" rpy=" 0 0 0"/>
+   <link name="caster_wheel">
+    <visual>
+      <origin xyz="0 0 0" rpy="0 0 0"/>
       <geometry>
-        <box size="${compute_length} ${compute_width} ${compute_height}"/>
-      </geometry>
-    </collision>
-    <visual name="chassis_visual">
-      <origin xyz="0 0 0" rpy=" 0 0 0"/>
-      <geometry>
-        <box size="${compute_length} ${compute_width} ${compute_height}"/>
+        <sphere radius="${caster_wheel_radius}"/>
       </geometry>
     </visual>
+    <collision>
+      <origin xyz="0 0 0" rpy="0 0 0"/>
+      <geometry>
+        <sphere radius="${caster_wheel_radius}"/>
+      </geometry>
+      <surface>
+            <friction>
+              <ode>
+                <mu>0.000000</mu>
+                <mu2>0.000000</mu2>
+                <slip1>1.000000</slip1>
+                <slip2>1.000000</slip2>
+              </ode>
+            </friction>
+          </surface>
+    </collision>
+    <xacro:sphere_inertia m="5" r="${caster_wheel_radius}"/>
   </link>
+  <joint name="caster_wheel_joint" type="continuous">
+    <axis xyz="0 1 0" rpy="0 0 0" />
+    <parent link="chassis"/>
+    <child link="caster_wheel"/>
+    <origin xyz="${caster_wheel_joint_offset} 0 -${caster_wheel_radius+chassis_height/2}" rpy="0 0 0"/>
+  </joint>
   <joint type="fixed" name="camera_joint">
     <origin xyz="${chassis_length/2 - camera_length} 0 ${chassis_height/2 + camera_height/2}" rpy="0 0 0"/>
@@ -186,18 +174,10 @@
   </joint>
   <joint type="fixed" name="hokuyo_joint">
-    <origin xyz="0 0 .02" rpy="0 0 0"/>
+    <origin xyz="0 0 0.06" rpy="0 0 0"/>
     <child link="hokuyo"/>
-    <parent link="compute"/>
-    <axis xyz="0 1 0" rpy="0 0 0"/>
-  </joint>
-  <joint type="fixed" name="compute_joint">
-    <origin xyz="-${compute_height/2} 0 ${chassis_height/2 + compute_height/2}" rpy="0 0 0"/>
-    <child link="compute"/>
     <parent link="chassis"/>
     <axis xyz="0 1 0" rpy="0 0 0"/>
   </joint>
-  <xacro:wheel fb="front" lr="right" parent="chassis" translateX="${wheel_base/2}" translateY="-${wheel_y_offset}"/>
-  <xacro:wheel fb="front" lr="left" parent="chassis" translateX="${wheel_base/2}" translateY="${wheel_y_offset}"/>
-  <xacro:wheel fb="back" lr="right" parent="chassis" translateX="-${wheel_base/2}" translateY="-${wheel_y_offset}"/>
-  <xacro:wheel fb="back" lr="left" parent="chassis" translateX="-${wheel_base/2}" translateY="${wheel_y_offset}"/>
+  <xacro:wheel lr="right" parent="chassis" translateX="${chassis_length/2-wheel_radius}" translateY="-${wheel_y_offset}"/>
+  <xacro:wheel lr="left" parent="chassis" translateX="${chassis_length/2-wheel_radius}" translateY="${wheel_y_offset}"/>
 </robot>

Commit message: feat: added depth camera

File: my_robot/urdf/my_robot.xacro (robot description, xacro)
@@ -179,4 +179,11 @@
     <axis xyz="0 1 0" rpy="0 0 0"/>
   </joint>
+  <joint name="camera_optical_joint" type="fixed">
+    <origin xyz="0 0 0" rpy="-1.5707 0 -1.5707"/>
+    <parent link="camera"/>
+    <child link="camera_link_optical"/>
+  </joint>
+  <link name="camera_link_optical">
+  </link>
   <xacro:wheel lr="right" parent="chassis" translateX="${chassis_length/2-wheel_radius}" translateY="-${wheel_y_offset}"/>
   <xacro:wheel lr="left" parent="chassis" translateX="${chassis_length/2-wheel_radius}" translateY="${wheel_y_offset}"/>
